Commit message: add imu publisher

File: go2w_description/urdf/go2w_description.urdf (robot description, URDF)
Before this commit: robot go2w_description, 33 links, 32 joints
Links:
- removed link base
- added link base_footprint
- added link base_link, mass 6.921; collision box size=0.3762 0.0935 0.114; visual mesh filename=package://go2w_description/dae/base.dae
- added link hesai_lidar, mass 0; collision cylinder length=0.08 radius=0.05; visual cylinder length=0.08 radius=0.05
Joints:
- added joint base_footprint_link: type fixed, parent base_footprint, child base_link, origin xyz=0 0 0.3 rpy=0 0 0
- added joint hesai_lidar_joint: type fixed, parent base_link, child hesai_lidar, origin xyz=0.145 0 0.11 rpy=0 0 0
- joint FL_hip_joint: parent base -> base_link
- joint FR_hip_joint: parent base -> base_link
- joint Head_upper_joint: parent base -> base_link
- joint RL_hip_joint: parent base -> base_link
- joint RR_hip_joint: parent base -> base_link
- joint imu_joint: parent base -> base_link
- joint radar_joint: parent base -> base_link

File: go2w_description/xacro/robot.xacro (robot description, xacro)
@@ -7,7 +7,7 @@
     <!-- Include base URDF -->
     <xacro:include filename="$(find go2w_description)/urdf/go2w_description.urdf"/>
-    <!-- Add XT16 Lidar if enabled -->
+    <!-- Add Hesai lidar frame if enabled -->
     <xacro:if value="$(arg add_lidar)">
-        <xacro:utlidar_sensor parent_link="base"/>
+        <xacro:hesai_lidar_sensor parent_link="base_link"/>
     </xacro:if>
 </robot>

File: go2w_description/xacro/sensors.xacro (robot description, xacro)
@@ -42,3 +42,30 @@
         </joint>
     </xacro:macro>
+    <!-- Hesai lidar frame compatible with go2_description -->
+    <xacro:macro name="hesai_lidar_sensor" params="parent_link">
+        <link name="hesai_lidar">
+            <inertial>
+                <origin xyz="0 0 0" rpy="0 0 0" />
+                <mass value="0" />
+                <inertia ixx="0" ixy="0" ixz="0" iyy="0" iyz="0" izz="0" />
+            </inertial>
+            <visual>
+                <origin xyz="0 0 0" rpy="0 0 0" />
+                <geometry>
+                    <cylinder radius="0.05" length="0.08" />
+                </geometry>
+            </visual>
+            <collision>
+                <origin xyz="0 0 0" rpy="0 0 0" />
+                <geometry>
+                    <cylinder radius="0.05" length="0.08" />
+                </geometry>
+            </collision>
+        </link>
+        <joint name="hesai_lidar_joint" type="fixed">
+            <origin xyz="0.145 0 0.11" rpy="0 0 0" />
+            <parent link="${parent_link}" />
+            <child link="hesai_lidar" />
+        </joint>
+    </xacro:macro>
 </robot>

Commit message: fix urdf hesai lidar

File: go2w_description/urdf/go2w_description.urdf (robot description, URDF)
Before this commit: robot go2w_description, 35 links, 34 joints
Joints:
- joint hesai_lidar_joint: origin xyz=0.145 0 0.11 rpy=0 0 0 -> xyz=0.145 0 0.11 rpy=0 0 1.57079632679

Commit message: add hesai lidar

File: go2w_description/urdf/go2w_description.urdf (robot description, URDF)
Before this commit: robot go2w_description, 35 links, 34 joints
Links:
- link hesai_lidar: geometry collision mesh filename=package://go2w_description/dae/XT32XT16.stl scale=0.001 0.001 0.001; visual mesh filename=package://go2w_description/dae/XT32XT16.stl scale=0.001 0.001 0.001

File: go2w_description/xacro/sensors.xacro (robot description, xacro)
@@ -51,13 +51,16 @@
             </inertial>
             <visual>
-                <origin xyz="0 0 0" rpy="0 0 0" />
+                <origin xyz="-0.00286 0 -0.025" rpy="1.5707963267948966 0 0" />
                 <geometry>
-                    <cylinder radius="0.05" length="0.08" />
+                    <mesh filename="package://go2w_description/dae/XT32XT16.stl" scale="0.001 0.001 0.001" />
                 </geometry>
+                <material name="hesai_lidar_material">
+                    <color rgba="0.20 0.22 0.24 1.0" />
+                </material>
             </visual>
             <collision>
-                <origin xyz="0 0 0" rpy="0 0 0" />
+                <origin xyz="-0.00286 0 -0.025" rpy="1.5707963267948966 0 0" />
                 <geometry>
-                    <cylinder radius="0.05" length="0.08" />
+                    <mesh filename="package://go2w_description/dae/XT32XT16.stl" scale="0.001 0.001 0.001" />
                 </geometry>
             </collision>

Commit message: merge imu and joint states publisher

File: go2w_description/urdf/go2w_description.urdf (robot description, URDF)
Before this commit: robot go2w_description, 35 links, 34 joints
Joints:
- joint hesai_lidar_joint: origin xyz=0.145 0 0.11 rpy=0 0 1.57079632679 -> xyz=0.145 0 0.11 rpy=0 0 0

Commit message: fix urdf

File: go2w_description/urdf/go2w_description.urdf (robot description, URDF)
Before this commit: robot go2w_description, 35 links, 34 joints
Joints:
- joint base_footprint_link: origin xyz=0 0 0.3 rpy=0 0 0 -> xyz=0 0 0.4 rpy=0 0 0
- joint hesai_lidar_joint: origin xyz=0.145 0 0.11 rpy=0 0 0 -> xyz=0.145 0 0.11 rpy=0 0 1.57079632679
