Commit message: add fast lio 2

File: go2w_description_modified/xacro/sensors.xacro (robot description, xacro)
@@ -29,5 +29,5 @@
             <child link="hesai_lidar" />
             <!-- Hesai LiDAR is mounted with a 90deg yaw rotation (per hardware). -->
-            <origin xyz="0.145 0 0.11" rpy="0 0 1.57079632679" />
+            <origin xyz="0.145 0 0.11" rpy="0 0 0" />
         </joint>
     </xacro:macro>
