Commit message: add fast lio2

File: go2w_description/xacro/go2w.xacro (robot description, xacro)
@@ -1,6 +1,6 @@
 <?xml version="1.0"?>
-<robot name="go2w_description_modified" xmlns:xacro="http://www.ros.org/wiki/xacro">
+<robot name="go2w_description" xmlns:xacro="http://www.ros.org/wiki/xacro">
     <!-- Import sensor definitions -->
-    <xacro:include filename="$(find go2w_description_modified)/xacro/sensors.xacro"/>
+    <xacro:include filename="$(find go2w_description)/xacro/sensors.xacro"/>
     <!-- Include original URDF from go2w_description (root link is "base") -->
     <xacro:include filename="$(find go2w_description)/urdf/go2w_description.urdf"/>

File: go2w_description/xacro/sensors.xacro (robot description, xacro)
@@ -12,5 +12,5 @@
                 <origin xyz="-0.00286 0 -0.025" rpy="1.5707963267948966 0 0" />
                 <geometry>
-                    <mesh filename="package://go2w_description_modified/stl/XT32XT16.stl" scale="0.001 0.001 0.001" />
+                    <mesh filename="package://go2w_description/stl/XT32XT16.stl" scale="0.001 0.001 0.001" />
                 </geometry>
                 <material name="hesai_lidar_material">
@@ -21,5 +21,5 @@
                 <origin xyz="-0.00286 0 -0.025" rpy="1.5707963267948966 0 0" />
                 <geometry>
-                    <mesh filename="package://go2w_description_modified/stl/XT32XT16.stl" scale="0.001 0.001 0.001" />
+                    <mesh filename="package://go2w_description/stl/XT32XT16.stl" scale="0.001 0.001 0.001" />
                 </geometry>
             </collision>

Commit message: add utlidar_lidar

File: go2w_description/xacro/go2w.xacro (robot description, xacro)
@@ -14,3 +14,10 @@
     <!-- Add Hesai LiDAR -->
     <xacro:hesai_lidar_sensor parent_link="base"/>
+    <!-- Add UTLidar frame, position matches radar while orientation matches base -->
+    <link name="utlidar_lidar" />
+    <joint name="utlidar_lidar_joint" type="fixed">
+        <origin xyz="0.28945 0 -0.046825" rpy="-2.924065656505679 -0.14998090081098114 -0.9763385649215685" />
+        <parent link="base" />
+        <child link="utlidar_lidar" />
+    </joint>
 </robot>
